Commit message: Commit new files

File: stereo_vision/launch/basic.urdf (robot description, URDF)
Before this commit: robot myfirst, 1 links, 0 joints
Links:
- added link stereo_cam; visual cylinder length=0.3 radius=0.05; visual cylinder length=0.3 radius=0.05
Joints:
- added joint usb_cam_to_stereo_cam: type fixed, parent usb_cam, child stereo_cam, origin xyz=0 0 1

Commit message: Modified rviz and urdf

File: stereo_vision/launch/basic.urdf (robot description, URDF)
Before this commit: robot handofros, 2 links, 1 joints
Links:
- added link left_camera; visual cylinder length=0.3 radius=0.05
- added link right_camera; visual cylinder length=0.3 radius=0.05
- link stereo_cam: geometry visual box size=0.1 0.2 0.1
Joints:
- added joint stereo_cam_to_left_camera: type fixed, parent stereo_cam, child left_camera, origin xyz=0.1 0.1 0
- added joint stereo_cam_to_right_camera: type fixed, parent stereo_cam, child right_camera, origin xyz=0.1 -0.1 0
